File: 1.Hardware/src/The_Girls'Gift.sch (KiCad schematic (older format))
At the start: 34 parts, among them J1 USB_B_Micro, Q1 AO3401A, SW1 Download, SW2 RESET, SW3 USER1, U1 CH551G, U2 662K, U3 LM75B, U4 4054, U5 MT3111

Commit message: master
Parts:
- removed D4, D5: LED, LED_SMD:LED_0603_1608Metric, symbol Device:LED
- removed R5, R6: R, Resistor_SMD:R_0603_1608Metric, symbol Device:R
- added H1: MountingHole, Common:Via_1.5, symbol Mechanical:MountingHole
- added TP1, TP2, TP3: TestPoint_Small, TestPoint:TestPoint_Pad_D1.0mm, symbol Connector:TestPoint_Small
- BT1: footprint (none) -> Battery:Battery_Li_8x9x3mm
- D1: footprint Diode_THT:D_DO-41_SOD81_P10.16mm_Horizontal -> Diode_SMD:D_SOD-323
- J1: footprint Connector_USB:USB_Micro-B_GCT_USB3076-30-A -> Connector_USB:USB_Micro-B_Molex-105017-0001
- SW1: footprint (none) -> Button_Switch_SMD:lfdcn_Button
- SW2: value RESET -> RST; footprint (none) -> Button_Switch_SMD:lfdcn_Button
- SW3: value USER1 -> USER; footprint (none) -> Button_Switch_SMD:lfdcn_Button
- U2: footprint Package_TO_SOT_SMD:TO-252-3_TabPin2 -> Package_TO_SOT_SMD:SOT-23
Connections:
- net +3V3: now also C8.2, SW1.1, SW2.1
- net GND: now also TP3.1
- net P30: now also TP2.1
- net P31: now also TP1.1
Other:
- moved on the sheet: U3
Changed lines of the file:
@@
 F 0 "J1" H 4635 4877 50  0000 R CNN
 F 1 "USB_B_Micro" H 4635 4968 50  0000 R CNN
-F 2 "Connector_USB:USB_Micro-B_GCT_USB3076-30-A" H 5015 4930 50  0001 C CNN
+F 2 "Connector_USB:USB_Micro-B_Molex-105017-0001" H 5015 4930 50  0001 C CNN
 F 3 "~" H 5015 4930 50  0001 C CNN
 	1    4865 4980
@@
 	4595 1150 4195 1150
 Connection ~ 4195 1150
-$Comp
-L Device:LED D4
-U 1 1 5FB47F63
-P 9390 3050
-F 0 "D4" H 9390 2870 50  0000 C CNN
-F 1 "LED" H 9390 2945 50  0000 C CNN
-F 2 "LED_SMD:LED_0603_1608Metric" H 9390 3050 50  0001 C CNN
-F 3 "~" H 9390 3050 50  0001 C CNN
-	1    9390 3050
-	-1   0    0    1
-$EndComp
-$Comp
-L Device:R R5
-U 1 1 5FB4831E
-P 9915 3050
-F 0 "R5" V 9708 3050 50  0000 C CNN
-F 1 "R" V 9799 3050 50  0000 C CNN
-F 2 "Resistor_SMD:R_0603_1608Metric" V 9845 3050 50  0001 C CNN
-F 3 "~" H 9915 3050 50  0001 C CNN
-	1    9915 3050
-	0    1    1    0
-$EndComp
-$Comp
-L Device:R R6
-U 1 1 5FB485F4
-P 9915 3400
-F 0 "R6" V 9708 3400 50  0000 C CNN
-F 1 "R" V 9799 3400 50  0000 C CNN
-F 2 "Resistor_SMD:R_0603_1608Metric" V 9845 3400 50  0001 C CNN
-F 3 "~" H 9915 3400 50  0001 C CNN
-	1    9915 3400
-	0    1    1    0
-$EndComp
-$Comp
-L Device:LED D5
-U 1 1 5FB4896A
-P 9390 3400
-F 0 "D5" H 9390 3200 50  0000 C CNN
-F 1 "LED" H 9390 3280 50  0000 C CNN
-F 2 "LED_SMD:LED_0603_1608Metric" H 9390 3400 50  0001 C CNN
-F 3 "~" H 9390 3400 50  0001 C CNN
-	1    9390 3400
-	-1   0    0    1
-$EndComp
-Wire Wire Line
-	9540 3050 9765 3050
-Wire Wire Line
-	9540 3400 9765 3400
-Wire Wire Line
-	10065 3050 10415 3050
-Wire Wire Line
-	10415 3050 10415 3400
-Wire Wire Line
-	10065 3400 10415 3400
-Connection ~ 10415 3400
-Wire Wire Line
-	10415 3400 10415 3500
-$Comp
-L power:GND #PWR030
-U 1 1 5FB4A818
-P 10415 3500
-F 0 "#PWR030" H 10415 3250 50  0001 C CNN
-F 1 "GND" H 10420 3327 50  0000 C CNN
-F 2 "" H 10415 3500 50  0001 C CNN
-F 3 "" H 10415 3500 50  0001 C CNN
-	1    10415 3500
-	1    0    0    -1
-$EndComp
-Wire Wire Line
-	9240 3050 8965 3050
-Wire Wire Line
-	9240 3400 8965 3400
 Text Label 3415 4880 0    50   ~ 0
 P37
@@
 F 0 "U2" H 2030 1367 50  0000 C CNN
 F 1 "662K" H 2030 1276 50  0000 C CNN
-F 2 "Package_TO_SOT_SMD:TO-252-3_TabPin2" H 2030 1050 50  0001 C CNN
+F 2 "Package_TO_SOT_SMD:SOT-23" H 2030 1050 50  0001 C CNN
 F 3 "https://static6.arrow.com/aropdfconversion/dc75757ae45a88e5f69bdce3f2a651a5fe0ca07d/ifx27001_ds_10.pdf" H 2030 1050 50  0001 C CNN
 	1    2030 1100
@@
 F 0 "BT1" H 5943 3131 50  0000 L CNN
 F 1 "Battery_3.7V" H 5943 3040 50  0000 L CNN
-F 2 "" V 5835 3145 50  0001 C CNN
+F 2 "Battery:Battery_Li_8x9x3mm" V 5835 3145 50  0001 C CNN
 F 3 "~" V 5835 3145 50  0001 C CNN
 	1    5835 3085
@@
 Text Label 11000 920  2    50   ~ 0
 P36
-$Comp
-L Switch:SW_Push SW2
-U 1 1 5FB5FAFC
-P 9160 1410
-F 0 "SW2" H 9160 1695 50  0000 C CNN
-F 1 "RESET" H 9160 1604 50  0000 C CNN
-F 2 "" H 9160 1610 50  0001 C CNN
-F 3 "~" H 9160 1610 50  0001 C CNN
-	1    9160 1410
-	1    0    0    -1
-$EndComp
-$Comp
-L Switch:SW_Push SW1
-U 1 1 5FB5F402
-P 9150 920
-F 0 "SW1" H 9150 1205 50  0000 C CNN
-F 1 "Download" H 9150 1114 50  0000 C CNN
-F 2 "" H 9150 1120 50  0001 C CNN
-F 3 "~" H 9150 1120 50  0001 C CNN
-	1    9150 920
-	1    0    0    -1
-$EndComp
-Text Label 8965 3050 0    50   ~ 0
-P30
-Text Label 8965 3400 0    50   ~ 0
-P31
 Wire Wire Line
 	9350 920  10225 920
@@
 F 0 "D1" V 2721 2675 50  0000 R CNN
 F 1 "1N5817" V 2630 2675 50  0000 R CNN
-F 2 "Diode_THT:D_DO-41_SOD81_P10.16mm_Horizontal" H 2675 2580 50  0001 C CNN
+F 2 "Diode_SMD:D_SOD-323" H 2675 2580 50  0001 C CNN
 F 3 "http://www.vishay.com/docs/88525/1n5817.pdf" H 2675 2755 50  0001 C CNN
 	1    2675 2755
@@
 	6060 1535 5695 1535
 Connection ~ 5695 1535
-$Comp
-L Switch:SW_Push SW3
-U 1 1 5FCED43E
-P 9835 2335
-F 0 "SW3" H 9835 2620 50  0000 C CNN
-F 1 "USER1" H 9835 2529 50  0000 C CNN
-F 2 "" H 9835 2535 50  0001 C CNN
-F 3 "~" H 9835 2535 50  0001 C CNN
-	1    9835 2335
-	1    0    0    -1
-$EndComp
 Wire Wire Line
 	10035 2335 10335 2335
@@
 L Sensor_Temperature:LM75B U3
 U 1 1 5FD4FA9E
-P 3275 6720
-F 0 "U3" H 3275 7401 50  0000 C CNN
-F 1 "LM75B" H 3275 7310 50  0000 C CNN
-F 2 "Package_SO:VSSOP-8_3.0x3.0mm_P0.65mm" H 3275 6720 50  0001 C CNN
-F 3 "http://www.ti.com/lit/ds/symlink/lm75b.pdf" H 3275 6720 50  0001 C CNN
-	1    3275 6720
+P 1465 6675
+F 0 "U3" H 1465 7356 50  0000 C CNN
+F 1 "LM75B" H 1465 7265 50  0000 C CNN
+F 2 "Package_SO:VSSOP-8_3.0x3.0mm_P0.65mm" H 1465 6675 50  0001 C CNN
+F 3 "http://www.ti.com/lit/ds/symlink/lm75b.pdf" H 1465 6675 50  0001 C CNN
+	1    1465 6675
 	1    0    0    -1
 $EndComp
@@
 L power:GND #PWR09
 U 1 1 5FD7F1BE
-P 3275 7330
-F 0 "#PWR09" H 3275 7080 50  0001 C CNN
-F 1 "GND" H 3275 7180 50  0000 C CNN
-F 2 "" H 3275 7330 50  0001 C CNN
-F 3 "" H 3275 7330 50  0001 C CNN
-	1    3275 7330
-	1    0    0    -1
-$EndComp
-Wire Wire Line
-	3275 7330 3275 7220
-Wire Wire Line
-	2875 6820 2670 6820
-Wire Wire Line
-	2875 6720 2670 6720
-Wire Wire Line
-	2875 6620 2670 6620
-Text Label 2670 6820 0    50   ~ 0
+P 1465 7285
+F 0 "#PWR09" H 1465 7035 50  0001 C CNN
+F 1 "GND" H 1465 7135 50  0000 C CNN
+F 2 "" H 1465 7285 50  0001 C CNN
+F 3 "" H 1465 7285 50  0001 C CNN
+	1    1465 7285
+	1    0    0    -1
+$EndComp
+Wire Wire Line
+	1465 7285 1465 7175
+Wire Wire Line
+	1065 6775 860  6775
+Wire Wire Line
+	1065 6675 860  6675
+Wire Wire Line
+	1065 6575 860  6575
+Text Label 860  6775 0    50   ~ 0
 P33
-Text Label 2670 6720 0    50   ~ 0
+Text Label 860  6675 0    50   ~ 0
 P14
-Text Label 2670 6620 0    50   ~ 0
+Text Label 860  6575 0    50   ~ 0
 P17
 Wire Wire Line
-	3275 6220 3275 5950
+	1465 6175 1465 5905
 $Comp
 L power:VCC #PWR08
 U 1 1 5FDAE42D
-P 3275 5950
-F 0 "#PWR08" H 3275 5800 50  0001 C CNN
-F 1 "VCC" V 3275 6070 50  0000 L CNN
-F 2 "" H 3275 5950 50  0001 C CNN
-F 3 "" H 3275 5950 50  0001 C CNN
-	1    3275 5950
-	1    0    0    -1
-$EndComp
-Wire Wire Line
-	3675 6620 3765 6620
-Wire Wire Line
-	3765 6620 3765 6720
-Wire Wire Line
-	3765 6720 3675 6720
-Wire Wire Line
-	3675 6820 3765 6820
-Wire Wire Line
-	3765 6820 3765 6720
-Connection ~ 3765 6720
-Wire Wire Line
-	3765 6820 3765 6950
-Connection ~ 3765 6820
-Text Label 3975 6950 2    50   ~ 0
+P 1465 5905
+F 0 "#PWR08" H 1465 5755 50  0001 C CNN
+F 1 "VCC" V 1465 6025 50  0000 L CNN
+F 2 "" H 1465 5905 50  0001 C CNN
+F 3 "" H 1465 5905 50  0001 C CNN
+	1    1465 5905
+	1    0    0    -1
+$EndComp
+Wire Wire Line
+	1865 6575 1955 6575
+Wire Wire Line
+	1955 6575 1955 6675
+Wire Wire Line
+	1955 6675 1865 6675
+Wire Wire Line
+	1865 6775 1955 6775
+Wire Wire Line
+	1955 6775 1955 6675
+Connection ~ 1955 6675
+Wire Wire Line
+	1955 6775 1955 6905
+Connection ~ 1955 6775
+Text Label 2165 6905 2    50   ~ 0
 P11
 Wire Wire Line
-	3765 6950 3975 6950
+	1955 6905 2165 6905
 Wire Notes Line
 	7580 4045 7580 470
@@
 $EndComp
 NoConn ~ 3415 5080
+$Comp
+L Switch:SW_Push SW1
+U 1 1 5FBD862D
+P 9150 920
+F 0 "SW1" H 9150 1205 50  0000 C CNN
+F 1 "Download" H 9150 1114 50  0000 C CNN
+F 2 "Button_Switch_SMD:lfdcn_Button" H 9150 1120 50  0001 C CNN
+F 3 "~" H 9150 1120 50  0001 C CNN
+	1    9150 920
+	1    0    0    -1
+$EndComp
+$Comp
+L Switch:SW_Push SW2
+U 1 1 5FBD9219
+P 9160 1410
+F 0 "SW2" H 9160 1695 50  0000 C CNN
+F 1 "RST" H 9160 1604 50  0000 C CNN
+F 2 "Button_Switch_SMD:lfdcn_Button" H 9160 1610 50  0001 C CNN
+F 3 "~" H 9160 1610 50  0001 C CNN
+	1    9160 1410
+	1    0    0    -1
+$EndComp
+$Comp
+L Switch:SW_Push SW3
+U 1 1 5FBD9A01
+P 9835 2335
+F 0 "SW3" H 9835 2620 50  0000 C CNN
+F 1 "USER" H 9835 2529 50  0000 C CNN
+F 2 "Button_Switch_SMD:lfdcn_Button" H 9835 2535 50  0001 C CNN
+F 3 "~" H 9835 2535 50  0001 C CNN
+	1    9835 2335
+	1    0    0    -1
+$EndComp
+$Comp
+L power:+3.3V #PWR0101
+U 1 1 5FC86D49
+P 8865 810
+F 0 "#PWR0101" H 8865 660 50  0001 C CNN
+F 1 "+3.3V" H 8750 940 50  0000 L CNN
+F 2 "" H 8865 810 50  0001 C CNN
+F 3 "" H 8865 810 50  0001 C CNN
+	1    8865 810
+	1    0    0    -1
+$EndComp
+Wire Wire Line
+	8865 810  8865 920
+Connection ~ 8865 920
+$Comp
+L Connector:TestPoint_Small TP1
+U 1 1 5FCA09F7
+P 3010 6000
+F 0 "TP1" H 3058 6046 50  0000 L CNN
+F 1 "TestPoint_Small" H 3058 5955 50  0000 L CNN
+F 2 "TestPoint:TestPoint_Pad_D1.0mm" H 3210 6000 50  0001 C CNN
+F 3 "~" H 3210 6000 50  0001 C CNN
+	1    3010 6000
+	1    0    0    -1
+$EndComp
+$Comp
+L Connector:TestPoint_Small TP2
+U 1 1 5FCA14D7
+P 3010 6180
+F 0 "TP2" H 3058 6226 50  0000 L CNN
+F 1 "TestPoint_Small" H 3058 6135 50  0000 L CNN
+F 2 "TestPoint:TestPoint_Pad_D1.0mm" H 3210 6180 50  0001 C CNN
+F 3 "~" H 3210 6180 50  0001 C CNN
+	1    3010 6180
+	1    0    0    -1
+$EndComp
+$Comp
+L Connector:TestPoint_Small TP3
+U 1 1 5FCA19BB
+P 3015 6350
+F 0 "TP3" H 3063 6396 50  0000 L CNN
+F 1 "TestPoint_Small" H 3063 6305 50  0000 L CNN
+F 2 "TestPoint:TestPoint_Pad_D1.0mm" H 3215 6350 50  0001 C CNN
+F 3 "~" H 3215 6350 50  0001 C CNN
+	1    3015 6350
+	1    0    0    -1
+$EndComp
+Text Label 2840 6000 0    50   ~ 0
+P31
+Wire Wire Line
+	2840 6000 3010 6000
+Wire Wire Line
+	3010 6180 2840 6180
+Text Label 2840 6180 0    50   ~ 0
+P30
+Wire Wire Line
+	3015 6350 2840 6350
+$Comp
+L power:GND #PWR0102
+U 1 1 5FCC23FE
+P 2840 6385
+F 0 "#PWR0102" H 2840 6135 50  0001 C CNN
+F 1 "GND" H 2840 6235 50  0000 C CNN
+F 2 "" H 2840 6385 50  0001 C CNN
+F 3 "" H 2840 6385 50  0001 C CNN
+	1    2840 6385
+	1    0    0    -1
+$EndComp
+Wire Wire Line
+	2840 6350 2840 6385
+$Comp
+L Mechanical:MountingHole H1
+U 1 1 5FC08262
+P 3405 6985
+F 0 "H1" H 3505 7031 50  0000 L CNN
+F 1 "MountingHole" H 3505 6940 50  0000 L CNN
+F 2 "Common:Via_1.5" H 3405 6985 50  0001 C CNN
+F 3 "~" H 3405 6985 50  0001 C CNN
+	1    3405 6985
+	1    0    0    -1
+$EndComp
 $EndSCHEMATC
