File: 1.Hardware/src/The_Girls'Gift.kicad_pcb (KiCad board)
At the start: 2 copper layers, 82 x 30 mm, 74 parts, among them J1 USB_B_Micro, Q1 AO3401A, SW1 Download, SW2 RST, SW3 USER, U1 CH551G, U2 662K, U3 LM75B, U4 4054, U5 MT3111

Commit message: master
Parts:
- removed the BT1 at (193.2, 80.4)
- removed the C1 at (213.6, 81.7)
- removed the C10 at (200.8, 86.9)
- removed the C2 at (213.5, 75.3)
- removed the C3 at (219.1, 82.1)
- removed the C4 at (213.5, 73.6)
- removed the C5 at (199.2, 84.6)
- removed the C6 at (211.7, 93.5)
- removed the C7 at (199.8, 73.2)
- removed the C8 at (198.8, 84.0)
- removed the C9 at (214.3, 84.1)
- removed the D1 at (195.5, 73.2)
- removed the D2 at (199.2, 87.0)
- removed the D3 at (207.1, 94.3)
- removed the G at (203.9, 87.1)
- removed the H1 at (207.0, 98.2)
- removed the J1 at (223.6, 79.9)
- removed the Q1 at (195.4, 81.5)
- removed the R at (201.8, 86.6)
- removed the R1 at (195.2, 76.9)
- removed the R2 at (195.3, 89.4)
- removed the R3 at (199.2, 89.4)
- removed the R4 at (199.2, 91.7)
- removed the R7 at (200.8, 89.6)
- removed the R8 at (214.3, 86.9)
- removed REF** (x6): Fiducial_0.5mm_Mask1mm, Fiducial:Fiducial_0.5mm_Mask1mm
- removed the SW1 at (207.1, 78.7)
- removed the SW2 at (199.8, 78.7)
- removed the SW3 at (214.3, 78.7)
- removed the T at (201.7, 84.3)
- removed the U1 at (207.0, 80.5)
- removed the U2 at (213.3, 77.9)
- removed the U3 at (207.0, 84.1)
- removed the U4 at (195.4, 85.7)
- removed the U5 at (207.1, 88.8)
Routing:
- net +5V: track 121.7 -> 60.9 mm, vias 4 -> 2
- net VCC: track 83.6 -> 41.8 mm, vias 6 -> 3
- net +3V3: track 58.6 -> 29.3 mm, vias 2 -> 1
- net /P36: track 58.3 -> 29.2 mm, vias 6 -> 3
- net GND: track 15.4 -> 0.00 mm, vias 12 -> 6
- net /P16: track 30.5 -> 15.2 mm, vias 2 -> 1
- net /P15: track 28.7 -> 14.3 mm, vias 2 -> 1
- net /P37: track 24.3 -> 12.1 mm
- net Net-(C9-Pad2): track 22.5 -> 11.2 mm
- net /P14: track 21.4 -> 10.7 mm, vias 2 -> 1
- net +BATT: track 21.1 -> 10.5 mm
- net /OUTB: track 20.3 -> 10.1 mm, vias 2 -> 1
- net /OUTG: track 19.8 -> 9.91 mm, vias 2 -> 1
- net /P32: track 19.4 -> 9.68 mm, vias 2 -> 1
- net /OUTR: track 18.4 -> 9.21 mm, vias 2 -> 1
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Other:
- board size 82 x 30 mm -> 40 x 30 mm
